File: hardware/kicad/ascii_stick_zero3_reiwa/ascii_stick_zero3_reiwa.kicad_pcb (KiCad board)
At the start: 2 copper layers, 69.3 x 65.3 mm, 19 parts, among them J1 USB_B_Micro, J2 Buttons_1, J3 AVR-ISP-6, J4 Buttons_2, J5 Buttons_3, J6 Buttons_4, J7 STICK, J8 STICK_POWER, U1 ATmega32U4-A, Y1 Crystal

Commit message: increase mergin of tracks from the MCU
Parts:
- moved J2 4.75 mm to (173.7, 113.8), turned to 90 degrees
- moved C3 4.50 mm to (184.8, 114.6)
- moved J6 3.91 mm to (189.9, 75.4)
- moved J5 3.80 mm to (205.3, 75.5)
Routing:
- net /BUTTON3: track 28.9 -> 21.4 mm
- net /BUTTON0: track 25.2 -> 29.2 mm
- net /BUTTON8: track 18.6 -> 14.8 mm
- net GND: track 192.3 -> 188.7 mm
- net /BUTTON2: track 27.2 -> 24.1 mm
- net /BUTTON13: track 10.4 -> 12.8 mm
- net /BUTTON9: track 16.3 -> 14.1 mm
- net Net-(U1-XTAL1): track 19.5 -> 21.3 mm
- net /BUTTON12: track 10.6 -> 12.1 mm
- net /BUTTON10: track 14.5 -> 13.4 mm
- net /BUTTON11: track 13.5 -> 12.7 mm
- net /BUTTON1: track 26.0 -> 26.7 mm
